File: cwm_.sch (EAGLE design)
At the start: 71 parts, among them U1 STM32L476, U2 24AA64T, U3 LSM9DS0, U4 MS5803-14BA, U5 MX25L25635F, U6 RN4020, U7 LTR-303ALS, U8 LM393, X1 EPSON FA-128 24.0000MF10Z-W3, X2 ABS06-32.768KHZ-9-1-T

Commit message: added all UCs
Parts:
- removed R14, R16, R18: 100k, resistor:R-EU_R0402
- removed R15, R17: 100R, resistor:R-EU_R0402
- removed T1, T2, T3: (no value), zetex:NMOSSOT23
- removed X2: ABS06-32.768KHZ-9-1-T, IQD-Frequency-Products:CRYSTALS-NOGND-IQXC-25
- added C11, C12: 1uF, resistor:C-EUC0603
- added C13: 10nF, resistor:C-EUC0603
- added U$3: NCP5623, NCP5623:NCP5623
- added U9: MK3200, MK3200:MK3200
- R10: value 5R -> 100k
- R13: value 100R -> 100k
- R8: value 5R -> 62k
- R9: value 60R -> 33R
- X1: value EPSON FA-128 24.0000MF10Z-W3 -> ABS06-32.768KHZ-9-1-T; device IQD-Frequency-Products:CRYSTALS-GND-LID-IQXC-42 -> IQD-Frequency-Products:CRYSTALS-NOGND-IQXC-25
Connections:
- removed net N$26: R17.1, R18.1, T1.G
- removed net N$27: R17.2
- net GND: now also C11.1, C12.2, C13.1, R8.2, S1.2, S3.2, U$3.GND1, U$3.GND2, U9.GND, U9.GND1, U9.PD; no longer R14.2, R16.2, R18.2, T1.S, T2.S, T3.S
- net N$11: now also U$3.LED2_G; no longer T1.D
- net N$12: now also LED1.BC, U$3.LED3_B; no longer LED1.RC, T2.D
- net N$13: now also LED1.RC, U$3.LED1_R; no longer LED1.BC, T3.D
- net N$19: now also U9.X1, X1.2; no longer R13.1, R14.1, T2.G
- net N$20: now also U$3.IREF; no longer LED1.GRN
- net N$21: now also U9.X2, X1.1; no longer LED1.RED, R9.1
- net N$22: now also R9.1, U9.OUT; no longer LED1.BLU, R10.1
- net N$23: now also U$1./RD; no longer R13.2
- net N$24: now also R10.2, S1.1; no longer R15.1, R16.1, T3.G
- net N$25: now also R13.1, S3.1; no longer R15.2
- net SCL: now also U$3.SCL
- net SDA: now also U$3.SDA
- net VCC: now also C13.2, R10.1, R13.2, U9.OE, U9.VDD; no longer R10.2, R8.2, R9.2, U$1./RD
- net VIN: now also C11.2, C12.1, LED1.BLU, LED1.GRN, LED1.RED, U$3.VBAT, U$3.VDET
Other:
- note removed: "Если будут ноги - повесить RD на IO"
- note removed: "Компараторы надо выключать - они целых 0.5мА жрут! каждый!"
- moved on the sheet: LED1, R10, R13, R8, R9

Commit message: some changes
Connections:
- new net N$26: R9.2, U1.PC14
- new net N$27: U6.UART_RX
- new net N$43: U6.UART_TX
- new net N$44: U6.RTS/PIO6
- new net N$45: U6.PIO5/CTS
- new net N$46: U6.CMD/MLDP
- new net N$47: U6.WAKE_SW
- new net N$48: U6.WAKE_HW
- new net N$49: U6.PIO1/SCK/PWM1
- new net N$50: U6.PIO2/CS/PWM2
- new net N$51: U6.PIO3/MOSI/PWM3
- new net N$53: U5.CS#
- new net N$54: U5.SO/SIO1
- new net N$55: U5.RESET#/SIO3
- new net N$56: U5.SCLK
- new net N$57: U5.SI/SIO0
- net GND: now also U1.VCAP1, U1.VCAP2, U6.GND, U6.GND1, U6.GND2, U6.GND3
- net N$23: now also U1.PH1
- net N$39: now also U1.PC15
- net N$5: now also U1.PC13
- net N$7: now also U1.PH0
- net SCL: now also U1.PC0
- net SDA: now also U1.PC1
- net VCC: now also U6.VDD
Other:
- note removed: "1-BURST, 0 - fixes"
- moved on the sheet: C8, C9, L1, PT1, PT3, R1, R11, R12, R20, R21, R23, R24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

Commit message: everything commected (draftely)
Parts:
- added R14, R15: 60k, resistor:R-EU_R0402
- C6: value 4.7uF - ceramic -> 4.7uF
Connections:
- removed net N$35: R22.2, U3.INT1(XM)
- removed net N$36: R19.2, U3.DRDY(G)
- removed net N$48: U6.WAKE_HW
- new net DRDY_G: R19.2, U1.PD2/SDIO_CMD, U3.DRDY(G)
- new net INT1_XM: R22.2, U1.PC12/SDIO_CLK, U3.INT1(XM)
- new net INT_LTR: R4.2, U1.PC2, U7.INT
- new net N$60: R14.2, R15.1, U1.PC3
- net GND: now also R14.1
- net N$16: now also U1.PA0
- net N$18: now also U1.PA1
- net N$23: now also U1.PA14/JTCK; no longer U1.PH1
- net N$24: now also U1.PC13
- net N$25: now also U1.PC5
- net N$27: now also U1.PA9/UART1_TX
- net N$41: now also U1.PC7
- net N$42: now also U1.PC8/SDIO_D0
- net N$43: now also U1.PA10/UART1_RX
- net N$44: now also U1.PA11
- net N$45: now also U1.PA12
- net N$46: now also U1.PC9/SDIO_D1
- net N$47: now also U1.PA8
- net N$49: now also U1.PC11/SDIO_D3
- net N$5: now also U1.PH1, U6.WAKE_HW; no longer R35.1, U$9.MODE/SYNC, U1.PC13
- net N$50: now also U1.PC10/SDIO_D2
- net N$51: now also U1.PA15/JTDI
- net N$53: now also U1.PA4/SPI1_NSS
- net N$54: now also U1.PA6/SPI1_MISO
- net N$55: now also U1.PC6/I2S2_MCK
- net N$56: now also U1.PA5/SPI1_SCK
- net N$57: now also U1.PA7/SPI1_MOSI
- net N$6: now also U1.PA3/UART2_RX
- net N$8: now also U1.PA2/UART2_TX
- net N$9: now also R35.1, U$9.MODE/SYNC, U1.PC4; no longer R4.2, U7.INT
- net VIN: now also R15.2
Other:
- note added: "добавить конденсаторы по питанию контроллера"
- note added: "посчитать правильные значения для резистивного делителя (чтобы максимальное напряжение было вольт 6)"
- note added: "уточнить корпуса для 10uF - просили алюминиевый по ДШ!"
- note removed: "уточнить корпуса для 0.22uF и 4.7uF и 10uF"
- moved on the sheet: C4, C8, C9, L1, R12, R2, R20, R21, R23, R24, R3, R35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
