File: cwm__.brd (EAGLE design)
At the start: 49.2 x 41.9 mm, 83 parts, among them U1 STM32L476, U2 24AA64T, U3 LSM9DS0, U4 MS5803-14BA, U5 MX25L25635F, U6 RN4020, U7 LTR-303ALS, U8 LM393, U9 MK3200, X1 ABS06-32.768KHZ-9-1-T

Commit message: first steps for routing
Parts:
- moved R4 55.4 mm to (48.8, 34.0), flipped to the bottom, turned to 90 degrees
- moved SV1 53.0 mm to (9.50, 41.0), turned to 180 degrees
- moved R2 52.8 mm to (37.5, 41.5)
- moved R38 50.5 mm to (33.8, 26.5), flipped to the bottom, turned to 270 degrees
- moved U7 50.4 mm to (47.0, 34.0), flipped to the bottom
- moved R17 50.3 mm to (19.5, 40.5), turned to 270 degrees
- moved C3 49.7 mm to (46.2, 31.5), flipped to the bottom
- moved R37 49.0 mm to (33.8, 29.5), flipped to the bottom, turned to 270 degrees
- moved R3 48.2 mm to (34.0, 41.5), turned to 0 degrees
- moved C11 47.8 mm to (47.0, 41.5), flipped to the bottom, turned to 0 degrees
- moved C18 47.3 mm to (16.5, 34.2), flipped to the bottom, turned to 90 degrees
- moved R8 46.5 mm to (47.0, 41.5), turned to 0 degrees
- moved C12 45.9 mm to (46.2, 34.8), turned to 0 degrees
- moved C21 45.6 mm to (19.5, 23.0), flipped to the bottom
- moved R16 42.2 mm to (25.2, 38.8), flipped to the bottom, turned to 90 degrees
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Connections:
- net VCC: no longer C20.2
- net VDD: now also C20.2
Other:
- board size 49.2 x 41.9 mm -> 50 x 42.9 mm

Commit message: routed version 0.1a
Parts:
- C13: device resistor:C0603 -> resistor:C0402
- T4: value (none) -> BSR202N L6327
- moved R18 7.75 mm to (32.8, 28.8), turned to 180 degrees
- moved R36 5.65 mm to (32.8, 26.4), turned to 0 degrees
- moved C10 2.35 mm to (34.8, 27.5)
- moved R38 2.21 mm to (36.0, 26.2)
- moved R37 2.20 mm to (36.0, 29.5)
- moved C20 1.62 mm to (32.8, 27.6), turned to 0 degrees
- moved C2 0.25 mm to (49.0, 32.0)
- moved R12 0.25 mm to (10.8, 27.5)
Routing:
- net GND: track 0.00 -> 373.6 mm, vias 0 -> 128
- net VCC: track 0.00 -> 292.2 mm, vias 0 -> 12
- net VIN: track 0.00 -> 73.5 mm, vias 0 -> 3
- net SCL: track 0.00 -> 62.3 mm, vias 0 -> 2
- net N$25: track 0.00 -> 55.0 mm
- net SDA: track 0.00 -> 53.8 mm, vias 0 -> 1
- net N$41: track 0.00 -> 50.8 mm, vias 0 -> 1
- net N$44: track 0.00 -> 47.9 mm, vias 0 -> 1
- net N$51: track 0.00 -> 45.5 mm, vias 0 -> 1
- net N$9: track 0.00 -> 43.0 mm
- net N$45: track 0.00 -> 41.4 mm, vias 0 -> 1
- net N$39: track 0.00 -> 38.1 mm, vias 0 -> 1
- net N$35: track 0.00 -> 37.9 mm
- net N$8: track 0.00 -> 36.8 mm, vias 0 -> 2
- net N$42: track 0.00 -> 36.7 mm, vias 0 -> 3
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- added copper zone on layer 1, net GND
- added copper zone on layer 16, net GND
Other:
- board text added: "CWM v0.1a"

Commit message: updated gerbers
Routing:
- net GND: track 373.6 -> 378.0 mm
Changed lines of the file:
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@@
 <setting verticaltext="up"/>
 </settings>
-<grid distance="0.5" unitdist="mm" unit="mm" style="lines" multiple="1" display="no" altdistance="0.025" altunitdist="inch" altunit="inch"/>
+<grid distance="0.05" unitdist="mm" unit="mm" style="lines" multiple="1" display="no" altdistance="0.025" altunitdist="inch" altunit="inch"/>
 <layers>
 <layer number="1" name="Top" color="4" fill="1" visible="yes" active="yes"/>
@@
 <attribute name="OC_NEWARK" value="unknown" x="10.75" y="25.25" size="1.778" layer="28" rot="MR0" display="off"/>
 <attribute name="MF" value="" x="10.75" y="25.25" size="1.778" layer="28" rot="MR0" display="off"/>
-<attribute name="VALUE" x="13.472" y="25.647" size="1.016" layer="28" ratio="10" rot="MR270"/>
+<attribute name="VALUE" x="14.472" y="25.647" size="1.016" layer="28" ratio="10" rot="MR270"/>
 </element>
 <element name="T5" library="zetex" package="SOT-23" value="" x="14.5" y="13.5" smashed="yes" rot="R270">
@@
 </element>
 <element name="U9" library="MK3200" package="SOIC8" value="MK3200" x="35.25" y="38" smashed="yes" rot="MR0">
-<attribute name="VALUE" x="38.032" y="37.559" size="1.016" layer="28" ratio="10" rot="MR0"/>
+<attribute name="VALUE" x="37.532" y="37.559" size="0.8" layer="28" ratio="10" rot="MR0"/>
 </element>
 <element name="R9" library="resistor" package="R0402" value="33R" x="32.25" y="33.5" smashed="yes" rot="MR270">
@@
 <wire x1="29.87173125" y1="3.46826875" x2="16.173" y2="3.46826875" width="0.254" layer="1"/>
 <wire x1="29.90673125" y1="3.50326875" x2="29.90673125" y2="4.62558125" width="0.254" layer="1"/>
-<wire x1="29.90673125" y1="4.62558125" x2="30.17815" y2="4.897" width="0.254" layer="1"/>
-<wire x1="30.17815" y1="4.897" x2="31.185840625" y2="4.897" width="0.254" layer="1"/>
-<wire x1="31.185840625" y1="4.897" x2="31.619759375" y2="5.33091875" width="0.254" layer="1"/>
+<wire x1="29.90673125" y1="4.62558125" x2="30.42815" y2="4.647" width="0.254" layer="1"/>
+<wire x1="30.42815" y1="4.647" x2="32.485840625" y2="4.647" width="0.4" layer="1"/>
+<wire x1="32.485840625" y1="4.647" x2="31.619759375" y2="5.33091875" width="0.254" layer="1"/>
 <wire x1="31.619759375" y1="5.33091875" x2="31.619759375" y2="12.404590625" width="0.254" layer="1"/>
 <wire x1="30.29" y1="3.12" x2="29.90673125" y2="3.50326875" width="0.254" layer="1"/>
@@
 <wire x1="49.125" y1="20.75" x2="49.125" y2="21.25" width="0.254" layer="16"/>
 <via x="24.461559375" y="18.762559375" extent="1-16" drill="0.4" diameter="0.6096"/>
-<wire x1="31.619759375" y1="12.404590625" x2="31.26885" y2="12.7555" width="0.254" layer="1"/>
-<wire x1="31.26885" y1="12.7555" x2="30.28858125" y2="12.7555" width="0.254" layer="1"/>
-<wire x1="30.28858125" y1="12.7555" x2="29.904290625" y2="13.139790625" width="0.254" layer="1"/>
-<wire x1="29.904290625" y1="13.139790625" x2="29.904290625" y2="14.234290625" width="0.254" layer="1"/>
-<wire x1="29.904290625" y1="14.234290625" x2="30.29" y2="14.62" width="0.254" layer="1"/>
+<wire x1="31.619759375" y1="12.404590625" x2="31.61885" y2="13.0555" width="0.254" layer="1"/>
+<wire x1="31.61885" y1="13.0555" x2="30.33858125" y2="13.0555" width="0.4" layer="1"/>
+<wire x1="30.33858125" y1="13.0555" x2="32.004290625" y2="13.089790625" width="0.4" layer="1"/>
+<wire x1="32.004290625" y1="13.089790625" x2="31.904290625" y2="14.234290625" width="0.254" layer="1"/>
+<wire x1="31.904290625" y1="14.234290625" x2="30.29" y2="14.62" width="0.254" layer="1"/>
 <wire x1="34.972990625" y1="25.6" x2="33.374190625" y2="24.0012" width="0.254" layer="16"/>
 <wire x1="33.374190625" y1="24.0012" x2="32.7394" y2="24.0012" width="0.254" layer="16"/>
@@
 <wire x1="27.662890625" y1="25.48911875" x2="28.04831875" y2="25.103690625" width="0.1524" layer="16"/>
 <wire x1="28.04831875" y1="25.103690625" x2="28.04831875" y2="18.464340625" width="0.1524" layer="16"/>
-<wire x1="28.04831875" y1="18.464340625" x2="27.41026875" y2="17.826290625" width="0.1524" layer="16"/>
-<wire x1="29.061390625" y1="11.87" x2="29.061390625" y2="16.17516875" width="0.1524" layer="1"/>
-<wire x1="29.061390625" y1="16.17516875" x2="27.41026875" y2="17.826290625" width="0.1524" layer="1"/>
+<wire x1="28.04831875" y1="18.464340625" x2="27.21026875" y2="17.626290625" width="0.1524" layer="16"/>
+<wire x1="29.061390625" y1="11.87" x2="29.061390625" y2="15.77516875" width="0.1524" layer="1"/>
+<wire x1="29.061390625" y1="15.77516875" x2="27.21026875" y2="17.626290625" width="0.1524" layer="1"/>
 <wire x1="30.29" y1="11.87" x2="29.061390625" y2="11.87" width="0.1524" layer="1"/>
-<via x="27.41026875" y="17.826290625" extent="1-16" drill="0.3048" diameter="0.6096"/>
+<via x="27.21026875" y="17.626290625" extent="1-16" drill="0.3048" diameter="0.6096"/>
 </signal>
 <signal name="N$50">
