File: cwm__.sch (EAGLE design)
At the start: 83 parts, among them U1 STM32L476, U2 24AA64T, U3 LSM9DS0, U4 MS5803-14BA, U5 MX25L25635F, U6 RN4020, U7 LTR-303ALS, U8 LM393, U9 MK3200, X1 ABS06-32.768KHZ-9-1-T

Commit message: first steps for routing
Connections:
- net VCC: no longer C20.2
- net VDD: now also C20.2
Changed lines of the file:
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@@
 <clearance class="1" value="0.2"/>
 </class>
-<class number="2" name="GND" width="0.254" drill="0.4">
+<class number="2" name="GND" width="0.3" drill="0.4">
 <clearance class="2" value="0.2"/>
 </class>
 <class number="3" name="VCC" width="0.254" drill="0.4">
 <clearance class="3" value="0.2"/>
+</class>
+<class number="4" name="VDD" width="0.254" drill="0.4">
+<clearance class="4" value="0.2"/>
 </class>
 </classes>
@@
 <part name="C19" library="resistor" deviceset="C-EU" device="C0402" value="100nF"/>
 <part name="GND48" library="SparkFun-Aesthetics" deviceset="GND" device=""/>
-<part name="SUPPLY47" library="SparkFun-Aesthetics" deviceset="VCC" device=""/>
 <part name="C20" library="resistor" deviceset="C-EU" device="C0402" value="100nF"/>
 <part name="GND49" library="SparkFun-Aesthetics" deviceset="GND" device=""/>
@@
 <part name="R37" library="resistor" deviceset="R-EU_" device="R0402" value="340k-1%"/>
 <part name="R38" library="resistor" deviceset="R-EU_" device="R0402" value="340k-1%"/>
+<part name="VDD3" library="supply1" deviceset="VDD" device=""/>
 </parts>
 <sheets>
@@
 <instance part="C19" gate="G$1" x="-294.64" y="149.86" rot="R180"/>
 <instance part="GND48" gate="1" x="-294.64" y="144.78"/>
-<instance part="SUPPLY47" gate="G$1" x="-320.04" y="175.26"/>
 <instance part="C20" gate="G$1" x="-320.04" y="170.18" rot="R180"/>
 <instance part="GND49" gate="1" x="-320.04" y="165.1"/>
@@
 <instance part="R37" gate="G$1" x="-226.06" y="55.88" rot="MR180"/>
 <instance part="R38" gate="G$1" x="-215.9" y="55.88" rot="MR180"/>
+<instance part="VDD3" gate="G$1" x="-320.04" y="177.8"/>
 </instances>
 <busses>
@@
 </segment>
 <segment>
-<pinref part="SUPPLY47" gate="G$1" pin="VCC"/>
-<pinref part="C20" gate="G$1" pin="2"/>
-</segment>
-<segment>
 <pinref part="SUPPLY48" gate="G$1" pin="VCC"/>
 <pinref part="C21" gate="G$1" pin="2"/>
@@
 <pinref part="R36" gate="G$1" pin="2"/>
 </segment>
-</net>
+<segment>
+<pinref part="C20" gate="G$1" pin="2"/>
+<pinref part="VDD3" gate="G$1" pin="VDD"/>
+</segment>
+</net>

Commit message: routed version 0.1a
Parts:
- C13: device resistor:C-EUC0603 -> resistor:C-EUC0402
- T4: value (none) -> BSR202N L6327
Changed lines of the file:
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@@
 <clearance class="1" value="0.2"/>
 </class>
-<class number="2" name="GND" width="0.3" drill="0.4">
+<class number="2" name="GND" width="0.254" drill="0.4">
 <clearance class="2" value="0.2"/>
 </class>
@@
 <part name="PT1" library="vishay_opto" deviceset="VEMT3700F" device=""/>
 <part name="S2" library="switch-reed" deviceset="REED-SWITCH-" device="MK15-C2"/>
-<part name="T4" library="zetex" deviceset="NMOSSOT23" device=""/>
+<part name="T4" library="zetex" deviceset="NMOSSOT23" device="" value="BSR202N L6327"/>
 <part name="T5" library="zetex" deviceset="NMOSSOT23" device=""/>
 <part name="S1" library="SparkFun-Electromechanical" deviceset="SWITCH-MOMENTARY-2" device="PTH"/>
@@
 <part name="SUPPLY37" library="SparkFun-Aesthetics" deviceset="VCC" device=""/>
 <part name="R9" library="resistor" deviceset="R-EU_" device="R0402" value="33R"/>
-<part name="C13" library="resistor" deviceset="C-EU" device="C0603" value="10nF"/>
+<part name="C13" library="resistor" deviceset="C-EU" device="C0402" value="10nF"/>
 <part name="GND33" library="SparkFun-Aesthetics" deviceset="GND" device=""/>
 <part name="R10" library="resistor" deviceset="R-EU_" device="R0402" value="100k"/>
